File: Main-DESKTOP-GF130J3.brd (EAGLE design)
At the start: 99 x 100 mm, 87 parts, among them IC1 UCC28180D, IC2 LTV-817-B, IC3 UCC24636DBVR, Q1 CSD19531Q5AT, Q2 IPA60R330P6XKSA1, Q3 IPA65R190CFD, T1 750311798, U1 TL431SOT23, X1 6ESRM-P

Commit message: Fix Cap Size v1
Parts:
- C1: device rcl:C0402K -> rcl:C0603
- CICOMP, CVCOMP2: device rcl:C0201 -> rcl:C0603K
- CISENSE: device rcl:C0201 -> rcl:C0402
- RFBB, RFREQ1, RGATE, RGATE1, RISENSE: device rcl:R0402 -> rcl:R0603
- RGATE2, RVCOMP: device rcl:R0201 -> rcl:R0603
- moved RFBB 255.1 mm to (158.8, 44.5)
- moved RGATE 255.1 mm to (151.1, 44.5)
- moved RVCOMP 255.1 mm to (106.7, 44.5)
- moved C1 255.1 mm to (129.5, 57.1)
- moved CICOMP 255.1 mm to (124.5, 44.5)
- moved CISENSE 255.1 mm to (144.8, 50.8)
- moved COUT 255.1 mm to (141.0, 66.0)
- moved COUTX 255.1 mm to (113.0, 57.1)
- moved CVCC 255.1 mm to (134.6, 35.6)
- moved CVCOMP 255.1 mm to (108.0, 50.8)
- moved CVSENSE 255.1 mm to (152.4, 57.1)
- moved DSTART 255.1 mm to (127.0, 66.0)
- moved DTURNOFF 255.1 mm to (143.5, 39.4)
- moved DZ 255.1 mm to (113.0, 64.8)
- moved IC1 255.1 mm to (127.0, 50.8)
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
Commit message: Cav Size v2
Parts:
- removed COUT: 5.435mF, cap-pan40:C10,0-14,0X6,0
- added C3, C6: (no value), Wurth_Elektronik_Passive_Capacitors_rev18b:30X10X2(DXPXΦ)
- moved DTURNOFF 131.0 mm to (12.7, 31.8), flipped to the bottom
- moved COUTX 47.6 mm to (128.3, 12.1)
- moved L2 22.8 mm to (67.3, 47.6)
- moved Q2 16.8 mm to (31.1, 38.1)
- moved CVCOMP2 9.44 mm to (14.0, 41.3)
- moved DBOOST 9.25 mm to (41.9, 38.1)
- moved RGATE2 6.63 mm to (12.7, 28.6), flipped to the bottom
- moved LBST 4.62 mm to (52.1, 50.2)
- moved CIN 1.91 mm to (87.6, 40.0)
- moved L6 1.42 mm to (93.3, 54.6)
- moved L5 1.27 mm to (81.3, 54.6)
- turned RFBT1 to 180 degrees
Connections:
- net GND: now also C3.2, C6.2; no longer COUT.2
- net VBULK: now also C3.1, C6.1; no longer COUT.1

Commit message: 090719
Parts:
- removed C6: (no value), Wurth_Elektronik_Passive_Capacitors_rev18b:30X10X2(DXPXΦ)
- added H1: CSM222-30AE, SamacSys_Parts:CSM22230AE
- added H2: HSE-B20250-040H-01, SamacSys_Parts:HSEB20250040H01
- added IC4: LM5021MM-1, SamacSys_Parts:SOP65P490X110-8N
- added IC5: UCC27714DR, SamacSys_Parts:SOIC127P600X175-14N
- added R15: WSK1206R0300FEA18, rcl:R3216
- added U2: HSE-B20254-035H, SamacSys_Parts:HSEB20254035H
- moved RFBB 192.8 mm to (-33.0, 65.3), flipped to the bottom, turned to 90 degrees
- moved RGATE 188.4 mm to (-36.4, 62.4), flipped to the bottom, turned to 180 degrees
- moved CVSENSE 187.3 mm to (-34.7, 65.2), flipped to the bottom, turned to 270 degrees
- moved RISENSE 179.3 mm to (-24.1, 58.9), flipped to the bottom
- moved CVCC 172.5 mm to (-36.3, 59.1), flipped to the bottom, turned to 0 degrees
- moved CISENSE 169.1 mm to (-24.2, 57.5), flipped to the bottom, turned to 180 degrees
- moved C1 165.7 mm to (-36.1, 60.7), flipped to the bottom
- moved IC1 157.2 mm to (-30.0, 59.0), flipped to the bottom
- moved C3 154.5 mm to (124.5, 4.95), turned to 180 degrees
- moved CICOMP 149.4 mm to (-24.1, 60.3), flipped to the bottom
- moved RFREQ1 144.2 mm to (-28.2, 55.5), flipped to the bottom
- moved CVCOMP 144.2 mm to (-36.1, 55.4), flipped to the bottom
- moved RVCOMP 139.9 mm to (-32.8, 55.4), flipped to the bottom
- moved DZ 136.1 mm to (-22.8, 55.6), flipped to the bottom, turned to 180 degrees
- moved RFB4 121.3 mm to (-2.54, -28.6)
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Connections:
- net N$12 renamed N$FREQ
- net N$13 renamed N$ISENSE
- net N$14 renamed N$VCOMP
- net N$29 renamed GATE
- net N$8 renamed N$ICOMP
- net N$9 renamed N$VSENSE
- removed net N$37: C4.2, F2.2, L3.2, R2.2, RV1.2
- new net N$9: IC5.1, IC5.2
- new net PH2: C4.1, F2.2, L3.2, R2.2, RV1.2
- new net VCC: IC4.3
- new net VSS: IC5.3
- net AGND: now also C1.2, CICOMP.1, CISENSE.2, CVCC.-, CVCOMP.2, CVCOMP2.1, CVSENSE.1, DZ.2, IC1.1, RFBB.2, RFREQ1.2
- net EMIOUT1: now also B2.AC2; no longer B2.AC1
- net EMIOUT2: now also B2.AC1; no longer B2.AC2
- net GND: now also IC4.5; no longer C3.2, C6.2, C8.2, COUTX.2, Q2.S, RGATE2.2, RSENSE.1
- net N$2: now also R15.1; no longer RSENSE.2
- net N$4: now also L5.2; no longer L5.1
- net N$40: now also C4.2; no longer C4.1
- net N$7: now also L5.1; no longer L5.2
- net PGND: now also C3.2, C8.2, COUTX.2, Q2.S, R15.2, RGATE2.2; no longer C1.2, CICOMP.1, CISENSE.2, CVCC.-, CVCOMP.2, CVCOMP2.1, CVSENSE.1, DZ.2, IC1.1, RFBB.2, RFREQ1.2
- net VBULK: no longer C6.1
- net VDD: now also IC5.7
Routing:
- net N$4: track 0.00 -> 197.5 mm
- net EMIOUT1: track 12.1 -> 116.5 mm
- net EMIOUT2: track 10.7 -> 107.8 mm
- net PH2: track 0.00 -> 80.3 mm
- net N$38: track 68.1 -> 142.9 mm
- net N$1: track 0.00 -> 70.1 mm
- net N$3: track 0.00 -> 52.5 mm
- net AGND: track 0.00 -> 47.8 mm
- net N$37: track 40.9 -> 0.00 mm
- net N$7: track 0.00 -> 36.3 mm
- net N$40: track 61.2 -> 92.5 mm
- net N$29: track 46.9 -> 70.2 mm
- net N$45: track 71.0 -> 50.9 mm
- net N$10: track 0.00 -> 9.64 mm
- net N$ISENSE: track 0.00 -> 8.64 mm
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
Commit message: 12 Juli 2019
Parts:
- removed D4: 1.5KE150A, SamacSys_Parts:DIOAD2920W106L900D505
- removed D5: STTH310S, SamacSys_Parts:DIOM8059X265N
- removed T1: 750311798, wurth_electronics_midcom_inc_v2-1:EE16/8/5_THT_H_9PIN_(5280)
- added D1: STTH310S, diode:SMC
- added DZ2: SMBJ130A-13-F, diode:SMBJ
- added T2: 750315800, SamacSys_Parts:PQ3230
- added T3: 750815330, wurth_electronics_midcom_inc_v2-1:EE25/13/7_THT_H_14PIN_(5644)
- moved Q1 151.9 mm to (9.53, 9.84)
- moved LS4 137.9 mm to (20.0, 9.21)
- moved CVCOMP 136.4 mm to (93.0, 11.4), turned to 270 degrees
- moved RFBB 136.4 mm to (90.9, 8.06), turned to 270 degrees
- moved CVSENSE 136.2 mm to (88.9, 8.00), turned to 90 degrees
- moved CVCOMP2 135.6 mm to (91.4, 11.3), turned to 90 degrees
- moved RVCOMP 132.2 mm to (93.0, 14.8), turned to 270 degrees
- moved RGATE 128.3 mm to (82.3, 13.7)
- moved CVCC 126.9 mm to (83.2, 16.3)
- moved C1 126.7 mm to (83.1, 18.0)
- moved IC1 126.5 mm to (89.5, 17.5), turned to 270 degrees
- moved RFREQ1 126.4 mm to (93.0, 19.4), turned to 270 degrees
- moved CISENSE 120.1 mm to (91.0, 23.4), turned to 90 degrees
- moved DZ 119.7 mm to (92.9, 24.8), turned to 90 degrees
- moved RISENSE 119.1 mm to (89.6, 23.4), turned to 270 degrees
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Connections:
- removed net AGND: C1.2, CDD1.-, CDD2.2, CICOMP.1, CISENSE.2, CLC.2, CVCC.-, CVCOMP.2, CVCOMP2.1, CVSENSE.1, DZ.2, IC1.1, L2.4, LS2.2, RFB4.1, RFBB.2, RFREQ1.2, RS2.1, T1.2
- removed net N$47: D7.1, RS1.2, T1.1
- new net N$12: D7.1, RS1.2, T3.6
- new net N$8: T3.3, T3.4
- net N$19: now also T3.12, T3.13; no longer T1.6
- net N$30: now also T3.10, T3.9; no longer T1.8
- net N$50: now also D1.C, DZ2.C; no longer D4.1, D5.1
- net N$52: now also D1.A, T3.2; no longer D5.2, T1.3
- net PGND: now also C1.2, CDD1.-, CDD2.2, CICOMP.1, CISENSE.2, CLC.2, CVCC.-, CVCOMP.2, CVCOMP2.1, CVSENSE.1, DZ.2, IC1.1, L2.4, LS2.2, RFB4.1, RFBB.2, RFREQ1.2, RS2.1, T3.7, U2.2
- net VBULK: now also DZ2.A, T3.5; no longer D4.2, T1.5
Routing:
- net PGND: track 3.61 -> 281.9 mm, vias 0 -> 11
- net VBULK: track 0.00 -> 136.9 mm, vias 0 -> 3
- net N$2: track 0.00 -> 75.6 mm
- net AGND: track 47.8 -> 0.00 mm
- net N$3: track 52.5 -> 22.4 mm
- net N$7: track 36.3 -> 62.3 mm
- net N$52: track 0.00 -> 25.9 mm
- net N$12: track 0.00 -> 25.4 mm, vias 0 -> 6
- net VCCCIC: track 7.16 -> 31.8 mm
- net N$VSENSE: track 0.00 -> 24.1 mm
- net N$29: track 70.2 -> 56.5 mm
- net N$31: track 0.00 -> 8.35 mm
- net N$11: track 0.00 -> 6.88 mm
- net N$1: track 70.1 -> 74.8 mm
- net EMIOUT1: track 116.5 -> 112.2 mm
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- added copper zone on layer 1, net N$12
- added copper zone on layer 16, net N$12
- added copper zone on layer 16, net N$2
- added copper zone on layer 1, net N$7
- added copper zone on layer 1, net PGND
- added copper zone on layer 16, net PGND
- added copper zone on layer 16, net VBULK

Commit message: Update Main-DESKTOP-GF130J3.brd
Routing:
- removed copper zone on layer 16, net N$12
Changed lines of the file:
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@@
 <contactref element="D7" pad="1"/>
 <contactref element="T3" pad="6"/>
-<wire x1="7.62" y1="45.72" x2="7.62" y2="33.9725" width="0.1524" layer="1"/>
-<wire x1="7.62" y1="33.9725" x2="9.8425" y2="31.75" width="0.1524" layer="1"/>
 <wire x1="9.68375" y1="31.90875" x2="9.8425" y2="31.75" width="0.1524" layer="1"/>
 <via x="9.8425" y="31.75" extent="1-16" drill="0.35" diameter="0.55" shape="octagon"/>
-<wire x1="9.8425" y1="31.75" x2="19.685" y2="31.75" width="0.1524" layer="16"/>
-<wire x1="19.685" y1="31.75" x2="20.0025" y2="31.4325" width="0.1524" layer="16"/>
-<wire x1="9.8425" y1="31.75" x2="-44.45" y2="-35.88" width="0" layer="19" extent="1-1"/>
-<wire x1="57.47" y1="-36.66" x2="20.0025" y2="31.4325" width="0" layer="19" extent="1-16"/>
 <polygon width="0.1524" layer="1">
 <vertex x="6.0325" y="45.72"/>
-<vertex x="6.35" y="46.0375"/>
-<vertex x="6.35" y="46.355"/>
+<vertex x="6.6675" y="46.355"/>
+<vertex x="6.6675" y="46.6725"/>
 <vertex x="6.985" y="46.99"/>
 <vertex x="8.255" y="46.99"/>
@@
 <vertex x="12.3825" y="33.655"/>
 <vertex x="13.0175" y="33.02"/>
-<vertex x="13.0175" y="32.0675"/>
 <vertex x="13.0175" y="30.1625"/>
 <vertex x="12.3825" y="29.5275"/>
 <vertex x="7.62" y="29.5275"/>
-<vertex x="6.35" y="30.7975"/>
 <vertex x="6.0325" y="31.115"/>
 <vertex x="6.0325" y="45.72"/>
 <vertex x="6.35" y="46.0375"/>
-</polygon>
-<polygon width="0.1524" layer="16">
-<vertex x="8.5725" y="32.7025"/>
-<vertex x="8.5725" y="33.3375"/>
-<vertex x="8.89" y="33.655"/>
-<vertex x="18.0975" y="33.655"/>
-<vertex x="18.415" y="33.3375"/>
-<vertex x="19.3675" y="32.385"/>
-<vertex x="19.3675" y="31.75"/>
-<vertex x="19.3675" y="30.1625"/>
-<vertex x="19.05" y="29.845"/>
-<vertex x="8.89" y="29.845"/>
-<vertex x="8.5725" y="30.1625"/>
 </polygon>
 <via x="9.8425" y="33.02" extent="1-16" drill="0.35" diameter="0.55" shape="octagon"/>
@@
 <via x="11.43" y="30.48" extent="1-16" drill="0.35" diameter="0.55" shape="octagon"/>
 <via x="9.8425" y="30.48" extent="1-16" drill="0.35" diameter="0.55" shape="octagon"/>
+<wire x1="7.62" y1="45.72" x2="7.62" y2="33.9725" width="2.54" layer="1"/>
+<wire x1="7.62" y1="33.9725" x2="9.8425" y2="31.75" width="2.54" layer="1"/>
+<wire x1="9.8425" y1="31.75" x2="19.685" y2="31.75" width="2.54" layer="16"/>
+<wire x1="19.685" y1="31.75" x2="20.0025" y2="31.4325" width="2.54" layer="16"/>
+<wire x1="9.8425" y1="30.48" x2="-44.45" y2="-35.88" width="0" layer="19" extent="1-1"/>
+<wire x1="9.8425" y1="31.75" x2="9.8425" y2="30.48" width="0" layer="19" extent="1-1"/>
+<wire x1="9.8425" y1="33.02" x2="9.68375" y2="31.90875" width="0" layer="19" extent="1-1"/>
+<wire x1="11.43" y1="33.02" x2="9.8425" y2="33.02" width="0" layer="19" extent="1-1"/>
+<wire x1="11.43" y1="31.75" x2="11.43" y2="33.02" width="0" layer="19" extent="1-1"/>
+<wire x1="11.43" y1="30.48" x2="11.43" y2="31.75" width="0" layer="19" extent="1-1"/>
+<wire x1="57.47" y1="-36.66" x2="20.0025" y2="31.4325" width="0" layer="19" extent="1-16"/>
 </signal>
 </signals>

Commit message: Update Main-DESKTOP-GF130J3.brd
Parts:
- moved RS2 140.9 mm to (76.8, 2.86), flipped to the bottom, turned to 270 degrees
- moved CDD1 139.6 mm to (67.6, 3.49), flipped to the bottom
- moved RCS1 128.8 mm to (67.9, 15.9), flipped to the bottom
- moved LS3 121.0 mm to (39.7, 21.6), flipped to the bottom, turned to 270 degrees
- moved CLC 118.9 mm to (72.7, 2.86), flipped to the bottom
- moved RLC 109.4 mm to (60.0, 18.7), flipped to the bottom, turned to 270 degrees
- moved U1 105.4 mm to (44.8, 19.7), flipped to the bottom, turned to 270 degrees
- moved LS1 105.3 mm to (50.8, 17.8), flipped to the bottom, turned to 270 degrees
- moved IC5 103.4 mm to (7.62, -24.1)
- moved RCS2 103.2 mm to (57.8, 18.7), flipped to the bottom
- moved R14 101.4 mm to (44.8, 16.8), flipped to the bottom, turned to 180 degrees
- moved R19 97.1 mm to (55.2, 19.1), flipped to the bottom
- moved R12 96.2 mm to (41.0, 16.8), flipped to the bottom, turned to 0 degrees
- moved R13 95.5 mm to (47.6, 17.8), flipped to the bottom
- moved R20 95.3 mm to (54.9, 23.2), flipped to the bottom, turned to 270 degrees
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Routing:
- net PGND: track 281.9 -> 428.5 mm, vias 11 -> 18
- net VDD: track 0.00 -> 125.0 mm, vias 0 -> 4
- net N$27: track 0.00 -> 103.8 mm, vias 0 -> 2
- net VOGND: track 0.00 -> 94.8 mm, vias 0 -> 4
- net N$30: track 0.00 -> 79.1 mm, vias 0 -> 3
- net N$19: track 0.00 -> 53.4 mm, vias 0 -> 4
- net N$42: track 0.00 -> 48.3 mm, vias 0 -> 6
- net N$12: track 25.4 -> 68.9 mm
- net N$22: track 0.00 -> 38.5 mm, vias 0 -> 1
- net N$46: track 0.00 -> 38.2 mm, vias 0 -> 2
- net N$52: track 25.9 -> 63.7 mm, vias 0 -> 3
- net N$17: track 0.00 -> 36.1 mm
- net VBULK: track 136.9 -> 172.8 mm, vias 3 -> 7
- net VCCCIC: track 31.8 -> 63.3 mm
- net N$15: track 0.00 -> 25.0 mm
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
Commit message: Update Main-DESKTOP-GF130J3.brd
Parts:
- moved LS4 1.59 mm to (18.4, 9.21)
- moved U2 1.14 mm to (44.8, 7.94)
- moved Q1 0.95 mm to (8.57, 9.84)
- moved CDD 0.64 mm to (18.1, 26.4)
- moved LS1 0.45 mm to (51.1, 18.1)
- moved R12 0.32 mm to (41.3, 16.8)
Routing:
- net N$40: track 77.5 -> 58.2 mm
- net N$52: track 63.7 -> 76.6 mm
- net VDD: track 125.0 -> 131.8 mm
- net N$29: track 56.5 -> 53.0 mm
- net N$19: track 53.4 -> 56.5 mm
- net N$27: track 103.8 -> 101.1 mm
- net N$46: track 38.2 -> 40.8 mm
- net PGND: track 428.5 -> 426.5 mm
- net N$22: track 38.5 -> 40.2 mm
- net VOGND: track 94.8 -> 93.4 mm, vias 4 -> 3
- net VBULK: track 172.8 -> 174.1 mm
- net N$50: track 17.0 -> 18.3 mm
- net N$26: track 18.3 -> 17.6 mm

Commit message: -
Parts:
- removed U2: HSE-B20254-035H, SamacSys_Parts:HSEB20254035H
- moved D7 51.5 mm to (8.89, 34.3)
- moved CLC 46.4 mm to (37.1, 32.7)
- moved CDD1 31.7 mm to (57.8, 33.7)
- moved RCS1 28.3 mm to (48.3, 36.2), turned to 270 degrees
- moved R1 27.3 mm to (31.1, 1.91)
- moved R5 27.0 mm to (37.5, 3.17)
- moved IC3 27.0 mm to (26.4, 2.86)
- moved R6 25.4 mm to (41.0, 4.13)
- moved RLC 24.7 mm to (39.7, 32.7)
- moved RCS2 21.4 mm to (45.4, 36.2), turned to 270 degrees
- moved IC2 20.3 mm to (33.3, 15.6)
- moved R11 20.1 mm to (44.8, 4.13)
- moved CFB3 18.7 mm to (59.1, 13.0)
- moved Q3 18.5 mm to (47.6, 27.9)
- moved R9 18.2 mm to (28.9, 5.40)
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Connections:
- net N$41 renamed N$DRV
- net N$42 renamed N$CS
- net N$46 renamed TOISENSE
- net PGND: no longer U2.2
Routing:
- net PGND: track 426.5 -> 290.2 mm, vias 18 -> 11
- net VDD: track 131.8 -> 0.32 mm, vias 4 -> 0
- net N$27: track 101.1 -> 0.00 mm, vias 2 -> 0
- net VOGND: track 93.4 -> 2.54 mm, vias 3 -> 0
- net N$30: track 79.2 -> 6.58 mm, vias 3 -> 0
- net N$12: track 68.9 -> 0.00 mm, vias 6 -> 0
- net N$19: track 56.5 -> 3.81 mm, vias 4 -> 0
- net VCCCIC: track 63.3 -> 16.9 mm
- net N$22: track 40.2 -> 0.00 mm, vias 1 -> 0
- net VBULK: track 174.1 -> 134.6 mm, vias 7 -> 5
- net N$17: track 36.1 -> 0.00 mm
- net N$CS: track 48.3 -> 13.0 mm, vias 6 -> 0
- net N$52: track 76.6 -> 46.1 mm, vias 3 -> 0
- net N$15: track 25.3 -> 0.00 mm
- net TOISENSE: track 40.8 -> 23.1 mm, vias 2 -> 0
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- removed copper zone on layer 1, net N$12
