File: Main-DESKTOP-GF130J3.brd (EAGLE design)
At the start: 99 x 100 mm, 93 parts, among them IC1 UCC28180D, IC2 LTV-817-B, IC3 UCC24636DBVR, IC4 LM5021MM-1, IC5 UCC27714DR, Q1 CSD19531Q5AT, Q2 IPA60R330P6XKSA1, Q3 IPA65R190CFD, T2 750315800, T3 750815330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

Commit message: 19 Juli
Parts:
- removed IC4: LM5021MM-1, SamacSys_Parts:SOP65P490X110-8N
- removed IC5: UCC27714DR, SamacSys_Parts:SOIC127P600X175-14N
- removed LS1: (no value), rcl:C0805
- removed R13, R14: (no value), rcl:R0805
- removed RSENSE: ERJ-L03KF50MV, ERJ-L03KF50MV:RC0603N
- removed T2: 750315800, SamacSys_Parts:PQ3230
- added 36: +36, con-wago-508:W237-4P
- added C2: (no value), rcl:C0603
- added C6: (no value), rcl:C0603K
- added COCOMP: (no value), rcl:C0805
- added ROFBB, ROFBT, ROPT: (no value), rcl:R0805
- R11: device rcl:R0805 -> rcl:R0603
- moved RS2 59.0 mm to (26.4, 33.3), turned to 0 degrees
- moved R11 45.6 mm to (1.27, -9.53), flipped to the top, turned to 0 degrees
- moved L2 35.8 mm to (12.7, 30.2), turned to 270 degrees
- moved CFB3 34.1 mm to (30.8, 32.1), turned to 180 degrees
- moved D1 26.4 mm to (59.1, 25.4), turned to 90 degrees
- moved R6 26.2 mm to (16.2, 12.7), turned to 0 degrees
- moved RFB3 22.0 mm to (30.8, 30.2)
- moved R1 21.1 mm to (15.2, 15.9)
- moved CDD1 20.1 mm to (38.1, 29.8), turned to 0 degrees
- moved R5 19.5 mm to (19.7, 11.1)
- moved U1 16.1 mm to (32.4, 12.7), turned to 180 degrees
- moved LS2 13.9 mm to (26.4, 31.1), turned to 180 degrees
- moved CDD2 13.1 mm to (20.3, 34.3), turned to 180 degrees
- moved C9 12.6 mm to (35.2, 33.7), flipped to the top
- moved LS3 12.0 mm to (16.2, 9.84), turned to 0 degrees
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Connections:
- net N$21 renamed N$VSC
- net N$23 renamed N$VPC
- net N$24 renamed N$TBK
- net N$26 renamed N$VODD
- removed net GND: IC4.5
- removed net N$9: IC5.1, IC5.2
- removed net VCC: IC4.3
- removed net VSS: IC5.3
- net N$15: now also ROPT.2; no longer R11.2
- net N$18: now also COCOMP.1, ROPT.1; no longer LS1.1, R11.1
- net N$19: now also 36.2, 36.4, ROFBT.2; no longer R13.2
- net N$5: now also COCOMP.2, ROFBB.2, ROFBT.1; no longer LS1.2, R13.1, R14.2
- net VDD: no longer IC5.7
- net VOGND: now also 36.1, 36.3, ROFBB.1; no longer R14.1
Routing:
- net VOGND: track 2.54 -> 147.5 mm, vias 0 -> 1
- net VCCCIC: track 16.9 -> 106.0 mm
- net N$19: track 3.81 -> 84.0 mm, vias 0 -> 2
- net PGND: track 290.2 -> 362.9 mm, vias 11 -> 15
- net VDD: track 0.32 -> 54.5 mm, vias 0 -> 2
- net N$30: track 6.58 -> 56.6 mm, vias 0 -> 1
- net N$DRV: track 5.95 -> 48.1 mm
- net N$17: track 0.00 -> 35.9 mm
- net N$50: track 3.37 -> 36.0 mm
- net N$52: track 46.1 -> 77.4 mm, vias 0 -> 1
- net N$CS: track 13.0 -> 43.1 mm
- net N$27: track 0.00 -> 26.9 mm
- net VBULK: track 134.6 -> 160.0 mm, vias 5 -> 3
- net N$12: track 0.00 -> 18.0 mm
- net N$VPC: track 0.00 -> 17.0 mm
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- added copper zone on layer 1, net VOGND
