File: Main-DESKTOP-GF130J3.sch (EAGLE design)
At the start: 87 parts, among them IC1 UCC28180D, IC2 LTV-817-B, IC3 UCC24636DBVR, Q1 CSD19531Q5AT, Q2 IPA60R330P6XKSA1, Q3 IPA65R190CFD, T1 750311798, U1 TL431SOT23, X1 6ESRM-P

Commit message: Fix Cap Size v1
Parts:
- C1: device rcl:C-EUC0402K -> rcl:C-EUC0603
- CICOMP, CVCOMP2: device rcl:C-EUC0201 -> rcl:C-EUC0603K
- CISENSE: device rcl:C-EUC0201 -> rcl:C-EUC0402
- RFBB, RFREQ1, RGATE, RGATE1, RISENSE: device rcl:R-EU_R0402 -> rcl:R-EU_R0603
- RGATE2, RVCOMP: device rcl:R-EU_R0201 -> rcl:R-EU_R0603
Changed lines of the file:
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@@
 <part name="COUT" library="cap-pan40" deviceset="C-NP" device="-10,0-14,0X6,0" value="5.435mF"/>
 <part name="DSTART" library="diode" library_urn="urn:adsk.eagle:library:210" deviceset="1N4446" device="" package3d_urn="urn:adsk.eagle:package:43344/2"/>
-<part name="RGATE1" library="rcl" library_urn="urn:adsk.eagle:library:334" deviceset="R-EU_" device="R0402" package3d_urn="urn:adsk.eagle:package:23547/3" value="1.07"/>
-<part name="RGATE2" library="rcl" library_urn="urn:adsk.eagle:library:334" deviceset="R-EU_" device="R0201" package3d_urn="urn:adsk.eagle:package:26117/2" value="10K"/>
+<part name="RGATE1" library="rcl" library_urn="urn:adsk.eagle:library:334" deviceset="R-EU_" device="R0603" package3d_urn="urn:adsk.eagle:package:23555/3" value="1.07"/>
+<part name="RGATE2" library="rcl" library_urn="urn:adsk.eagle:library:334" deviceset="R-EU_" device="R0603" package3d_urn="urn:adsk.eagle:package:23555/3" value="10K"/>
 <part name="IC1" library="SamacSys_Parts" deviceset="UCC28180D" device=""/>
 <part name="PGND" library="supply1" library_urn="urn:adsk.eagle:library:371" deviceset="GND" device="" value="PGND"/>
 <part name="CVSENSE" library="rcl" library_urn="urn:adsk.eagle:library:334" deviceset="C-EU" device="C0805" package3d_urn="urn:adsk.eagle:package:23617/2" value="820nF"/>
-<part name="CICOMP" library="rcl" library_urn="urn:adsk.eagle:library:334" deviceset="C-EU" device="C0201" package3d_urn="urn:adsk.eagle:package:23690/2" value="1.5nF"/>
-<part name="RISENSE" library="rcl" library_urn="urn:adsk.eagle:library:334" deviceset="R-EU_" device="R0402" package3d_urn="urn:adsk.eagle:package:23547/3" value="221"/>
+<part name="CICOMP" library="rcl" library_urn="urn:adsk.eagle:library:334" deviceset="C-EU" device="C0603K" package3d_urn="urn:adsk.eagle:package:23680/2" value="1.5nF"/>
+<part name="RISENSE" library="rcl" library_urn="urn:adsk.eagle:library:334" deviceset="R-EU_" device="R0603" package3d_urn="urn:adsk.eagle:package:23555/3" value="221"/>
 <part name="VBULK" library="supply2" library_urn="urn:adsk.eagle:library:372" deviceset="VPP" device=""/>
-<part name="RFREQ1" library="rcl" library_urn="urn:adsk.eagle:library:334" deviceset="R-EU_" device="R0402" package3d_urn="urn:adsk.eagle:package:23547/3" value="17.4K"/>
+<part name="RFREQ1" library="rcl" library_urn="urn:adsk.eagle:library:334" deviceset="R-EU_" device="R0603" package3d_urn="urn:adsk.eagle:package:23555/3" value="17.4K"/>
 <part name="L5" library="Wurth_Elektronik_Passive_rev18f" library_urn="urn:adsk.eagle:library:7584915" deviceset="WE-FI" device="_7447016" package3d_urn="urn:adsk.eagle:package:7586765/3"/>
 <part name="L6" library="Wurth_Elektronik_Passive_rev18f" library_urn="urn:adsk.eagle:library:7584915" deviceset="WE-FI" device="_7447016" package3d_urn="urn:adsk.eagle:package:7586765/3"/>
 <part name="DBOOST" library="diode" library_urn="urn:adsk.eagle:library:210" deviceset="DIODE-" device="TO220V" package3d_urn="urn:adsk.eagle:package:43373/3" value="LXA06T600"/>
 <part name="Q2" library="transistor-power" library_urn="urn:adsk.eagle:library:400" deviceset="PMOSFET_N" device="TO220BV" package3d_urn="urn:adsk.eagle:package:29484/3" value="IPA60R330P6XKSA1"/>
-<part name="CISENSE" library="rcl" library_urn="urn:adsk.eagle:library:334" deviceset="C-EU" device="C0201" package3d_urn="urn:adsk.eagle:package:23690/2" value="1nF"/>
+<part name="CISENSE" library="rcl" library_urn="urn:adsk.eagle:library:334" deviceset="C-EU" device="C0402" package3d_urn="urn:adsk.eagle:package:23626/2" value="1nF"/>
 <part name="CVCOMP" library="rcl" library_urn="urn:adsk.eagle:library:334" deviceset="C-EU" device="C0805" package3d_urn="urn:adsk.eagle:package:23617/2" value="22uF"/>
 <part name="SUPPLY2" library="supply2" library_urn="urn:adsk.eagle:library:372" deviceset="GND" device="" value="PGND"/>
 <part name="DTURNOFF" library="SamacSys_Parts" deviceset="MBR0540T1G" device=""/>
-<part name="RFBB" library="rcl" library_urn="urn:adsk.eagle:library:334" deviceset="R-EU_" device="R0402" package3d_urn="urn:adsk.eagle:package:23547/3" value="13K"/>
-<part name="RGATE" library="rcl" library_urn="urn:adsk.eagle:library:334" deviceset="R-EU_" device="R0402" package3d_urn="urn:adsk.eagle:package:23547/3" value="3.92"/>
-<part name="C1" library="rcl" library_urn="urn:adsk.eagle:library:334" deviceset="C-EU" device="C0402K" package3d_urn="urn:adsk.eagle:package:23679/2" value="100nF"/>
+<part name="RFBB" library="rcl" library_urn="urn:adsk.eagle:library:334" deviceset="R-EU_" device="R0603" package3d_urn="urn:adsk.eagle:package:23555/3" value="13K"/>
+<part name="RGATE" library="rcl" library_urn="urn:adsk.eagle:library:334" deviceset="R-EU_" device="R0603" package3d_urn="urn:adsk.eagle:package:23555/3" value="3.92"/>
+<part name="C1" library="rcl" library_urn="urn:adsk.eagle:library:334" deviceset="C-EU" device="C0603" package3d_urn="urn:adsk.eagle:package:23616/2" value="100nF"/>
 <part name="RSENSE" library="ERJ-L03KF50MV" deviceset="ERJ-L03KF50MV" device=""/>
 <part name="RFBT" library="CRCW2512300KJNEG" deviceset="CRCW2512300KJNEG" device=""/>
 <part name="RFBT1" library="CRCW2512300KJNEG" deviceset="CRCW2512300KJNEG" device=""/>
 <part name="RFBT2" library="CRCW2512402KFKEG" deviceset="CRCW2512402KFKEG" device=""/>
-<part name="CVCOMP2" library="rcl" library_urn="urn:adsk.eagle:library:334" deviceset="C-EU" device="C0201" package3d_urn="urn:adsk.eagle:package:23690/2" value="22nF"/>
-<part name="RVCOMP" library="rcl" library_urn="urn:adsk.eagle:library:334" deviceset="R-EU_" device="R0201" package3d_urn="urn:adsk.eagle:package:26117/2" value="287K"/>
+<part name="CVCOMP2" library="rcl" library_urn="urn:adsk.eagle:library:334" deviceset="C-EU" device="C0603K" package3d_urn="urn:adsk.eagle:package:23680/2" value="22nF"/>
+<part name="RVCOMP" library="rcl" library_urn="urn:adsk.eagle:library:334" deviceset="R-EU_" device="R0603" package3d_urn="urn:adsk.eagle:package:23555/3" value="287K"/>
 <part name="COUTX" library="cap-pan40" deviceset="C-NP" device="-10,0-14,0X6,0" value="100nF"/>
 <part name="DZ" library="TZMC1V0-M-18" deviceset="TZMC1V0-M-18" device="" package3d_urn="urn:adsk.eagle:package:11886536/1"/>

Commit message: Cav Size v2
Parts:
- removed COUT: 5.435mF, cap-pan40:C-NP-10,0-14,0X6,0
- added C3, C6: (no value), Wurth_Elektronik_Passive_Capacitors_rev18b:WCAP-AIG8_30X46_861011485018
Connections:
- net GND: now also C3.2, C6.2; no longer COUT.2
- net VBULK: now also C3.1, C6.1; no longer COUT.1
Changed lines of the file:
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@@
 <part name="Q1" library="SamacSys_Parts" deviceset="CSD19531Q5AT" device=""/>
 <part name="LBST" library="Wurth_Elektronik_Passive_rev18f" library_urn="urn:adsk.eagle:library:7584915" deviceset="WE-SI" device="_744139" package3d_urn="urn:adsk.eagle:package:7586520/3" value="494.23uH"/>
-<part name="COUT" library="cap-pan40" deviceset="C-NP" device="-10,0-14,0X6,0" value="5.435mF"/>
 <part name="DSTART" library="diode" library_urn="urn:adsk.eagle:library:210" deviceset="1N4446" device="" package3d_urn="urn:adsk.eagle:package:43344/2"/>
 <part name="RGATE1" library="rcl" library_urn="urn:adsk.eagle:library:334" deviceset="R-EU_" device="R0603" package3d_urn="urn:adsk.eagle:package:23555/3" value="1.07"/>
@@
 <part name="CIN" library="rcl" library_urn="urn:adsk.eagle:library:334" deviceset="C-EU" device="150-072X183" package3d_urn="urn:adsk.eagle:package:23657/1" value="890283325008CS"/>
 <part name="B2" library="rectifier" library_urn="urn:adsk.eagle:library:336" deviceset="GBU4" device="" package3d_urn="urn:adsk.eagle:package:23875/1"/>
+<part name="C3" library="Wurth_Elektronik_Passive_Capacitors_rev18b" library_urn="urn:adsk.eagle:library:491551" deviceset="WCAP-AIG8" device="_861011485018" package3d_urn="urn:adsk.eagle:package:491739/2" technology="_30X46"/>
+<part name="C6" library="Wurth_Elektronik_Passive_Capacitors_rev18b" library_urn="urn:adsk.eagle:library:491551" deviceset="WCAP-AIG8" device="_861011485018" package3d_urn="urn:adsk.eagle:package:491739/2" technology="_30X46"/>
 </parts>
 <sheets>
@@
 <attribute name="VALUE" x="55.88" y="88.9" size="1.778" layer="96"/>
 </instance>
-<instance part="COUT" gate="G$1" x="132.08" y="76.2" smashed="yes" rot="R270">
-<attribute name="NAME" x="127.635" y="78.74" size="1.778" layer="95" rot="R270"/>
-<attribute name="VALUE" x="135.636" y="80.9625" size="1.778" layer="96" rot="R270"/>
-</instance>
 <instance part="DSTART" gate="1" x="73.66" y="101.6" smashed="yes">
 <attribute name="NAME" x="76.2" y="102.0826" size="1.778" layer="95"/>
@@
 <attribute name="NAME" x="10.16" y="93.98" size="1.778" layer="95"/>
 <attribute name="VALUE" x="10.16" y="87.63" size="1.778" layer="96"/>
+</instance>
+<instance part="C3" gate="G$1" x="132.08" y="73.66" smashed="yes">
+<attribute name="NAME" x="135.255" y="78.74" size="1.778" layer="95"/>
+<attribute name="VALUE" x="135.255" y="70.485" size="1.778" layer="96"/>
+</instance>
+<instance part="C6" gate="G$1" x="142.24" y="73.66" smashed="yes">
+<attribute name="NAME" x="145.415" y="78.74" size="1.778" layer="95"/>
+<attribute name="VALUE" x="145.415" y="70.485" size="1.778" layer="96"/>
 </instance>
 </instances>
@@
 <pinref part="DSTART" gate="1" pin="C"/>
 <wire x1="76.2" y1="101.6" x2="132.08" y2="101.6" width="0.1524" layer="91"/>
-<pinref part="COUT" gate="G$1" pin="1"/>
 <wire x1="132.08" y1="78.74" x2="132.08" y2="91.44" width="0.1524" layer="91"/>
 <wire x1="116.84" y1="91.44" x2="132.08" y2="91.44" width="0.1524" layer="91"/>
@@
 <pinref part="RFBT2" gate="A" pin="1"/>
 <wire x1="170.18" y1="91.44" x2="170.18" y2="88.9" width="0.1524" layer="91"/>
+<pinref part="C3" gate="G$1" pin="1"/>
+<junction x="132.08" y="78.74"/>
+<pinref part="C6" gate="G$1" pin="1"/>
+<wire x1="142.24" y1="78.74" x2="132.08" y2="78.74" width="0.1524" layer="91"/>
 </segment>
 </net>
@@
 <net name="GND" class="0">
 <segment>
-<pinref part="COUT" gate="G$1" pin="2"/>
-<wire x1="132.08" y1="55.88" x2="132.08" y2="73.66" width="0.1524" layer="91"/>
+<wire x1="132.08" y1="55.88" x2="132.08" y2="71.12" width="0.1524" layer="91"/>
 <wire x1="116.84" y1="55.88" x2="132.08" y2="55.88" width="0.1524" layer="91"/>
 <pinref part="PGND" gate="1" pin="GND"/>
@@
 <pinref part="COUTX" gate="G$1" pin="2"/>
 <wire x1="152.4" y1="55.88" x2="152.4" y2="73.66" width="0.1524" layer="91"/>
-</segment>
-</net>
+<junction x="132.08" y="71.12"/>
+<pinref part="C3" gate="G$1" pin="2"/>
+<junction x="132.08" y="71.12"/>
+<pinref part="C6" gate="G$1" pin="2"/>
+<wire x1="132.08" y1="71.12" x2="142.24" y2="71.12" width="0.1524" layer="91"/>
+</segment>
+</net>

Commit message: 090719
Parts:
- removed C6: (no value), Wurth_Elektronik_Passive_Capacitors_rev18b:WCAP-AIG8_30X46_861011485018
- added H1: CSM222-30AE, SamacSys_Parts:CSM222-30AE
- added H2: HSE-B20250-040H-01, SamacSys_Parts:HSE-B20250-040H-01
- added IC4: LM5021MM-1, SamacSys_Parts:LM5021MM-1
- added IC5: UCC27714DR, SamacSys_Parts:UCC27714DR
- added R15: WSK1206R0300FEA18, rcl:R-EU_R3216
- added U2: HSE-B20254-035H, SamacSys_Parts:HSE-B20254-035H
Connections:
- net N$12 renamed N$FREQ
- net N$13 renamed N$ISENSE
- net N$14 renamed N$VCOMP
- net N$29 renamed GATE
- net N$8 renamed N$ICOMP
- net N$9 renamed N$VSENSE
- removed net GND: C3.2, C6.2, C8.2, COUTX.2, Q2.S, RGATE2.2, RSENSE.1
- removed net N$37: C4.2, F2.2, L3.4, R2.2, RV1.2
- new net N$9: IC5.HI, IC5.LI
- new net PH2: C4.1, F2.2, L3.4, R2.2, RV1.2
- net AGND: now also C1.2, CICOMP.1, CISENSE.2, CVCC.-, CVCOMP.2, CVCOMP2.1, CVSENSE.1, DZ.C, IC1.GND, RFBB.2, RFREQ1.2
- net EMIOUT1: now also B2.AC1; no longer B2.AC2
- net EMIOUT2: now also B2.AC2; no longer B2.AC1
- net N$2: now also R15.1; no longer RSENSE.2
- net N$4: now also L5.2; no longer L5.1
- net N$40: now also C4.2; no longer C4.1
- net N$7: now also L5.1; no longer L5.2
- net PGND: now also C3.2, C8.2, COUTX.2, Q2.S, R15.2, RGATE2.2; no longer C1.2, CICOMP.1, CISENSE.2, CVCC.-, CVCOMP.2, CVCOMP2.1, CVSENSE.1, DZ.C, IC1.GND, RFBB.2, RFREQ1.2
- net VBULK: no longer C6.1
Other:
- moved on the sheet: C4, L5

Commit message: 12 Juli 2019
Parts:
- removed D4: 1.5KE150A, SamacSys_Parts:1.5KE150A
- removed D5: STTH310S, SamacSys_Parts:STTH310S
- removed T1: 750311798, wurth_electronics_midcom_inc_v2-1:750311798
- added D1: STTH310S, diode:DIODE-SMC
- added DZ2: SMBJ130A-13-F, diode:SUPPRESSOR-SMBJ
- added T2: 750315800, SamacSys_Parts:750315800
- added T3: 750815330, wurth_electronics_midcom_inc_v2-1:750815330
Connections:
- removed net AGND: C1.2, CDD1.-, CDD2.2, CICOMP.1, CISENSE.2, CLC.2, CVCC.-, CVCOMP.2, CVCOMP2.1, CVSENSE.1, DZ.C, IC1.GND, L2.GND, LS2.2, RFB4.1, RFBB.2, RFREQ1.2, RS2.1, T1.2
- removed net N$47: D7.P$1, RS1.2, T1.1
- new net N$12: D7.P$1, RS1.2, T3.6
- new net N$8: T3.3, T3.4
- net N$19: now also T3.12, T3.13; no longer T1.6
- net N$30: now also T3.10, T3.9; no longer T1.8
- net N$50: now also D1.C, DZ2.C; no longer D4.K, D5.K
- net N$52: now also D1.A, T3.2; no longer D5.A, T1.3
- net PGND: now also C1.2, CDD1.-, CDD2.2, CICOMP.1, CISENSE.2, CLC.2, CVCC.-, CVCOMP.2, CVCOMP2.1, CVSENSE.1, DZ.C, IC1.GND, L2.GND, LS2.2, RFB4.1, RFBB.2, RFREQ1.2, RS2.1, T3.7, U2.2
- net VBULK: now also DZ2.A, T3.5; no longer D4.A, T1.5
Other:
- moved on the sheet: C1, CDD1, CDD2, LS2, RFB4, RS2

Commit message: -
Parts:
- removed U2: HSE-B20254-035H, SamacSys_Parts:HSE-B20254-035H
Connections:
- net N$41 renamed N$DRV
- net N$42 renamed N$CS
- net N$46 renamed TOISENSE
- net PGND: no longer U2.2
Other:
- moved on the sheet: RCS1, RCS2
Changed lines of the file:
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@@
 <part name="H1" library="SamacSys_Parts" deviceset="CSM222-30AE" device=""/>
 <part name="H2" library="SamacSys_Parts" deviceset="HSE-B20250-040H-01" device=""/>
-<part name="U2" library="SamacSys_Parts" deviceset="HSE-B20254-035H" device=""/>
 <part name="IC4" library="SamacSys_Parts" deviceset="LM5021MM-1" device=""/>
 <part name="IC5" library="SamacSys_Parts" deviceset="UCC27714DR" device="" override_package3d_urn="urn:adsk.eagle:package:12025919/2" override_package_urn="urn:adsk.eagle:footprint:12025920/1" override_locally_modified="yes"/>
@@
 <attribute name="NAME" x="107.95" y="68.58" size="1.778" layer="95" align="center-left"/>
 <attribute name="VALUE" x="113.03" y="68.58" size="1.778" layer="96" align="center-left"/>
-</instance>
-<instance part="U2" gate="G$1" x="121.92" y="43.18" smashed="yes">
-<attribute name="NAME" x="138.43" y="50.8" size="1.778" layer="95" align="center-left"/>
-<attribute name="VALUE" x="138.43" y="48.26" size="1.778" layer="96" align="center-left"/>
 </instance>
 <instance part="FRAME2" gate="G$1" x="-91.44" y="-78.74" smashed="yes">
@@
 <pinref part="R15" gate="G$1" pin="2"/>
 <wire x1="63.5" y1="48.26" x2="58.42" y2="48.26" width="0.1524" layer="91"/>
-<wire x1="132.08" y1="55.88" x2="132.08" y2="43.18" width="0.1524" layer="91"/>
 <junction x="132.08" y="-10.16"/>
-<pinref part="U2" gate="G$1" pin="2"/>
-<wire x1="132.08" y1="43.18" x2="132.08" y2="-10.16" width="0.1524" layer="91"/>
-<junction x="132.08" y="43.18"/>
+<wire x1="132.08" y1="55.88" x2="132.08" y2="-10.16" width="0.1524" layer="91"/>
 <pinref part="Q2" gate="G$1" pin="S"/>
 <wire x1="99.314" y1="68.199" x2="99.06" y2="65.659" width="0.1524" layer="91"/>
@@
 <attribute name="VALUE" x="-6.096" y="63.881" size="1.778" layer="96"/>
 </instance>
-<instance part="RCS1" gate="G$1" x="96.52" y="66.04" smashed="yes" rot="R90">
-<attribute name="NAME" x="95.0214" y="62.23" size="1.778" layer="95" rot="R90"/>
-<attribute name="VALUE" x="99.822" y="62.23" size="1.778" layer="96" rot="R90"/>
+<instance part="RCS1" gate="G$1" x="99.06" y="66.04" smashed="yes" rot="R90">
+<attribute name="NAME" x="97.5614" y="62.23" size="1.778" layer="95" rot="R90"/>
+<attribute name="VALUE" x="102.362" y="62.23" size="1.778" layer="96" rot="R90"/>
 </instance>
 <instance part="RS1" gate="G$1" x="-2.54" y="86.36" smashed="yes" rot="R90">
@@
 <attribute name="VALUE" x="92.71" y="74.422" size="1.778" layer="96" rot="R180"/>
 </instance>
-<instance part="RCS2" gate="G$1" x="101.6" y="66.04" smashed="yes" rot="R90">
-<attribute name="NAME" x="100.1014" y="62.23" size="1.778" layer="95" rot="R90"/>
-<attribute name="VALUE" x="104.902" y="62.23" size="1.778" layer="96" rot="R90"/>
+<instance part="RCS2" gate="G$1" x="104.14" y="66.04" smashed="yes" rot="R90">
+<attribute name="NAME" x="102.6414" y="62.23" size="1.778" layer="95" rot="R90"/>
+<attribute name="VALUE" x="107.442" y="62.23" size="1.778" layer="96" rot="R90"/>
 </instance>
 <instance part="R19" gate="G$1" x="96.52" y="78.74" smashed="yes" rot="R90">
@@
 </segment>
 </net>
-<net name="N$41" class="0">
+<net name="N$DRV" class="0">
 <segment>
 <pinref part="L2" gate="G$1" pin="DRV"/>
@@
 </segment>
 </net>
-<net name="N$46" class="0">
+<net name="TOISENSE" class="0">
 <segment>
 <pinref part="R19" gate="G$1" pin="1"/>
 <pinref part="RCS1" gate="G$1" pin="2"/>
-<wire x1="96.52" y1="73.66" x2="96.52" y2="71.12" width="0.1524" layer="91"/>
+<wire x1="96.52" y1="73.66" x2="99.06" y2="71.12" width="0.1524" layer="91"/>
 <pinref part="RLC" gate="G$1" pin="1"/>
-<wire x1="96.52" y1="71.12" x2="93.98" y2="71.12" width="0.1524" layer="91"/>
-<junction x="96.52" y="71.12"/>
+<wire x1="99.06" y1="71.12" x2="93.98" y2="71.12" width="0.1524" layer="91"/>
+<junction x="99.06" y="71.12"/>
 <pinref part="RCS2" gate="G$1" pin="2"/>
-<wire x1="101.6" y1="71.12" x2="96.52" y2="71.12" width="0.1524" layer="91"/>
+<wire x1="104.14" y1="71.12" x2="99.06" y2="71.12" width="0.1524" layer="91"/>
 <pinref part="Q3" gate="G$1" pin="S"/>
-<wire x1="101.6" y1="71.12" x2="104.14" y2="71.12" width="0.1524" layer="91"/>
 <wire x1="104.14" y1="71.12" x2="104.14" y2="81.28" width="0.1524" layer="91"/>
-<junction x="101.6" y="71.12"/>
-</segment>
-</net>
-<net name="N$42" class="0">
+<junction x="104.14" y="71.12"/>
+</segment>
+</net>
+<net name="N$CS" class="0">
 <segment>
 <pinref part="RLC" gate="G$1" pin="2"/>
@@
 <pinref part="RCS2" gate="G$1" pin="1"/>
 <pinref part="RCS1" gate="G$1" pin="1"/>
-<wire x1="101.6" y1="60.96" x2="96.52" y2="60.96" width="0.1524" layer="91"/>
-<wire x1="81.28" y1="60.96" x2="96.52" y2="60.96" width="0.1524" layer="91"/>
+<wire x1="104.14" y1="60.96" x2="99.06" y2="60.96" width="0.1524" layer="91"/>
+<wire x1="81.28" y1="60.96" x2="99.06" y2="60.96" width="0.1524" layer="91"/>
 <junction x="81.28" y="60.96"/>
-<junction x="96.52" y="60.96"/>
+<junction x="99.06" y="60.96"/>
 <pinref part="L2" gate="G$1" pin="GND"/>
 <wire x1="33.02" y1="71.12" x2="34.29" y2="71.12" width="0.1524" layer="91"/>
