File: Main-DCDC Only.sch (EAGLE design)
At the start: 93 parts, among them IC1 UCC28180D, IC2 LTV-817-B, IC3 UCC24636DBVR, Q1 CSD19531Q5AT, Q2 IPA60R330P6XKSA1, Q3 IPA65R190CFD, T3 750815330, U1 TL431SOT23, X1 6ESRM-P

Commit message: 19 Juli
Parts:
- removed B2: (no value), rectifier:GBU4
- removed C1: 100nF, rcl:C-EUC0603
- removed C2: (no value), rcl:C-EUC0603
- removed C3: (no value), Wurth_Elektronik_Passive_Capacitors_rev18b:WCAP-AIG8_30X46_861011485018
- removed C6: (no value), rcl:C-EUC0603K
- removed CICOMP: 1.5nF, rcl:C-EUC0603K
- removed CIN: 890283325008CS, rcl:C-EU150-072X183
- removed CISENSE: 1nF, rcl:C-EUC0402
- removed COUTX: 100nF, cap-pan40:C-NP-10,0-14,0X6,0
- removed CVCC: 293D105X9025A2TE3, rcl:CPOL-EUCT3216
- removed CVCOMP: 22uF, rcl:C-EUC0805
- removed CVCOMP2: 22nF, rcl:C-EUC0603K
- removed CVSENSE: 820nF, rcl:C-EUC0805
- removed DBOOST: LXA06T600, diode:DIODE-TO220V
- removed DSTART: 1N4446, diode:1N4446
- removed DTURNOFF: MBR0540T1G, SamacSys_Parts:MBR0540T1G
- removed DZ: TZMC1V0-M-18, TZMC1V0-M-18:TZMC1V0-M-18
- removed H1: CSM222-30AE, SamacSys_Parts:CSM222-30AE
- removed H2: HSE-B20250-040H-01, SamacSys_Parts:HSE-B20250-040H-01
- removed IC1: UCC28180D, SamacSys_Parts:UCC28180D
- removed L5, L6: (no value), Wurth_Elektronik_Passive_rev18f:WE-FI_7447016
- removed LBST: 494.23uH, Wurth_Elektronik_Passive_rev18f:WE-SI_744139
- removed Q2: IPA60R330P6XKSA1, transistor-power:PMOSFET_NTO220BV
- removed R11: (no value), rcl:R-EU_R0603
- removed R15: WSK1206R0300FEA18, rcl:R-EU_R3216
- removed RFBB: 13K, rcl:R-EU_R0603
- removed RFBT, RFBT1: CRCW2512300KJNEG, CRCW2512300KJNEG:CRCW2512300KJNEG
- removed RFBT2: CRCW2512402KFKEG, CRCW2512402KFKEG:CRCW2512402KFKEG
- removed RFREQ1: 17.4K, rcl:R-EU_R0603
- removed RGATE: 3.92, rcl:R-EU_R0603
- removed RGATE1: 1.07, rcl:R-EU_R0603
- removed RGATE2: 10K, rcl:R-EU_R0603
- removed RISENSE: 221, rcl:R-EU_R0603
- removed RVCOMP: 287K, rcl:R-EU_R0603
Connections:
- removed net GATE: IC1.GATE, RGATE.2
- removed net N$1: B2.-, L6.1
- removed net N$10: DTURNOFF.A, Q2.G, RGATE1.2, RGATE2.1
- removed net N$11: DTURNOFF.K, RGATE.1, RGATE1.1
- removed net N$16: CVCOMP.1, RVCOMP.2
- removed net N$2: CIN.2, L6.2, R15.1, RISENSE.1
- removed net N$28: RFBT1.1, RFBT2.2
- removed net N$3: DBOOST.A, LBST.2, Q2.D
- removed net N$31: RFBT.1, RFBT1.2
- removed net N$4: B2.+, L5.2
- removed net N$7: CIN.1, DSTART.A, L5.1, LBST.1
- removed net N$FREQ: IC1.FREQ, RFREQ1.1
- removed net N$ICOMP: CICOMP.2, IC1.ICOMP
- removed net N$ISENSE: CISENSE.1, DZ.A, IC1.ISENSE, RISENSE.2
- removed net N$VCOMP: CVCOMP2.2, IC1.VCOMP, RVCOMP.1
- removed net N$VSENSE: CVSENSE.2, IC1.VSENSE, RFBB.1, RFBT.2
- net EMIOUT1: no longer B2.AC1
- net EMIOUT2: no longer B2.AC2
- net PGND: no longer C1.2, C3.2, CICOMP.1, CISENSE.2, COUTX.2, CVCC.-, CVCOMP.2, CVCOMP2.1, CVSENSE.1, DZ.C, IC1.GND, Q2.S, R15.2, RFBB.2, RFREQ1.2, RGATE2.2
- net VBULK: no longer C3.1, COUTX.1, DBOOST.C, DSTART.C, RFBT2.1
- net VCCCIC: no longer C1.1, CVCC.+, IC1.VCC
